File: waterleak V.1.kicad_pcb (KiCad board)
At the start: 2 copper layers, 29 x 31 mm, 16 parts, among them J1 Conn_01x03_Pin, J2 waterleak sensor, Q2 MMBT2222A, U2 LM358

Commit message: add gerber
Connections:
- net +3.3V renamed +5V
Changed lines of the file:
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@@
 			(outputformat 1)
 			(mirror no)
-			(drillshape 1)
+			(drillshape 0)
 			(scaleselection 1)
-			(outputdirectory "")
+			(outputdirectory "waterleak gerber/")
 		)
 	)
 	(net 0 "")
-	(net 1 "+3.3V")
+	(net 1 "+5V")
 	(net 2 "GND")
 	(net 3 "Net-(J2-Pin_1)")
@@
 			(layers "F.Cu" "F.Paste" "F.Mask")
 			(roundrect_rratio 0.25)
-			(net 1 "+3.3V")
+			(net 1 "+5V")
 			(pinfunction "V+")
 			(pintype "power_in")
@@
 			(layers "F.Cu" "F.Paste" "F.Mask")
 			(roundrect_rratio 0.212766)
-			(net 1 "+3.3V")
+			(net 1 "+5V")
 			(pintype "passive")
 		)
@@
 			(layers "F.Cu" "F.Paste" "F.Mask")
 			(roundrect_rratio 0.208333)
-			(net 1 "+3.3V")
+			(net 1 "+5V")
 			(pintype "passive")
 		)
@@
 			(layers "*.Cu" "*.Mask")
 			(remove_unused_layers no)
-			(net 1 "+3.3V")
+			(net 1 "+5V")
 			(pinfunction "1")
 			(pintype "passive")
@@
 			(layers "*.Cu" "*.Mask")
 			(remove_unused_layers no)
-			(net 1 "+3.3V")
+			(net 1 "+5V")
 			(pinfunction "Pin_1")
 			(pintype "passive")
@@
 	)
 	(segment
+		(start 75.2 64.16)
+		(end 75.56 63.8)
+		(width 0.6)
+		(layer "F.Cu")
+		(net 1)
+	)
+	(segment
 		(start 93.1 68.8)
 		(end 93.1 73.9)
@@
 		(layer "F.Cu")
 		(net 1)
-	)
-	(segment
-		(start 75.2 64.16)
-		(end 75.56 63.8)
-		(width 0.6)
-		(layer "F.Cu")
-		(net 1)
